File: hardware/arinc429.kicad_pcb (KiCad board)
At the start: 2 copper layers, 40 x 60 mm, 60 parts, among them P1 CON-SENSOR2, P2 BOOT, P3 DEBUG, P4 IND 8Pol, U1 XMC1404, U2 DRILL, U3 DRILL, U4 DRILL, U5 DRILL, U6 HI-3593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

Commit message: edited F.Paste layer
Other:
- board text added: "D1, D2, D4, D5, D6, D7 not in F.Paste Layer!!"

Commit message: added specific partnumber HI-3593PQIF
Parts:
- U6: value HI-3593 -> HI-3593PQIF
Changed lines of the file:
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@@
       (effects (font (size 1 1) (thickness 0.15)))
     )
-    (fp_text value HI-3593 (at 0 2.65 270) (layer F.Fab)
+    (fp_text value HI-3593PQIF (at 0 2.65 270) (layer F.Fab)
       (effects (font (size 1 1) (thickness 0.15)))
     )
